Commit message: Modifica file principali per integrazione con il robot

File: soft_robotics/soft_robotics_description/urdf/soft_robotics_description_macro.xacro (robot description, xacro)
@@ -1,16 +1,13 @@
 <?xml version="1.0"?>
-<robot name="soft_robotics_gripper" xmlns:xacro="http://www.ros.org/wiki/xacro">
-  <material name="Grey">
-    <color rgba="0.2 0.2 0.2 1" />
-  </material>
-  <material name="Blue">
-    <color rgba="0 0 1 1" />
-  </material>
-  <xacro:macro name="soft_robotics_gripper" params="prefix parent *origin">
-    <joint name="soft_robotics_gripper_base_joint" type="fixed">
-      <origin xyz="0 0 -0.15" rpy=" 0 0 ${pi/2}" />
-      <parent link="tool0" />
-      <child link="soft_robotics_gripper_base_link" />
-    </joint>
+<robot xmlns:xacro="http://www.ros.org/wiki/xacro">
+  <xacro:macro name="soft_robotics_description" params="prefix">
+    <xacro:include filename="$(find soft_robotics_description)/urdf/soft_robotics_transmission.xacro" />
+    <xacro:soft_robotics_transmission prefix="${prefix}"/>
+    <material name="Grey">
+      <color rgba="0.2 0.2 0.2 1" />
+    </material>
+    <material name="Blue">
+      <color rgba="0 0 1 1" />
+    </material>
     <link name="soft_robotics_gripper_base_link">
       <visual>
@@ -131,38 +128,4 @@
       </inertial>
     </link>
-  <gazebo reference="soft_robotics_gripper_base_link">
-        <material>Gazebo/Grey</material>
-  </gazebo>
-  <gazebo reference="soft_robotics_left_finger_link1">
-        <material>Gazebo/Blue</material>
-  </gazebo>
-  <gazebo reference="soft_robotics_right_finger_link1">
-        <material>Gazebo/Blue</material>
-  </gazebo>
-    <gazebo reference="soft_robotics_left_finger_link2">
-        <material>Gazebo/Blue</material>
-  </gazebo>
-  <gazebo reference="soft_robotics_right_finger_link2">
-        <material>Gazebo/Blue</material>
-  </gazebo>
-    <!-- TRANSMISSION -->
-    <transmission name="right_finger_trans">
-      <type>transmission_interface/SimpleTransmission</type>
-      <joint name="soft_robotics_gripper_left_finger_joint1">
-        <hardwareInterface>hardware_interface/PositionJointInterface</hardwareInterface>
-      </joint>
-      <actuator name="right_finger_motor">
-        <mechanicalReduction>1</mechanicalReduction>
-      </actuator>
-    </transmission>
-    <transmission name="left_finger_trans">
-      <type>transmission_interface/SimpleTransmission</type>
-      <joint name="soft_robotics_gripper_right_finger_joint1">
-        <hardwareInterface>hardware_interface/PositionJointInterface</hardwareInterface>
-      </joint>
-      <actuator name="${prefix}shoulder_lift_motor">
-        <mechanicalReduction>1</mechanicalReduction>
-      </actuator>
-    </transmission>
   </xacro:macro>
 </robot>
