Commit message: Modifiche movimento, planning e miglioramento delle performance di MoveIt

File: UR5e_gripper/integration_package/urdf/ur5e_gripper.xacro (robot description, xacro)
@@ -66,5 +66,5 @@
   <!-- Attach gripper to robot arm -->
   <joint name="soft_robotics_gripper_base_joint" type="fixed">
-    <origin xyz="0 0 0" rpy=" 0 0 ${-pi/2}" />
+    <origin xyz="0 0 0" rpy=" 0 0 ${pi/2}" />
     <parent link="tool0" />
     <child link="soft_robotics_gripper_base_link" />

Commit message: Modifiche configurazione robot e mondo

File: UR5e_gripper/integration_package/urdf/ur5e_gripper.xacro (robot description, xacro)
@@ -62,5 +62,5 @@
     <parent link="world"/>
     <child link="base_link"/>
-    <origin xyz="0 0 1.79" rpy="${-pi} 0 0"/>
+    <origin xyz="0 0 1.79" rpy="${-pi} 0 ${pi}"/>
   </joint>
   <!-- Attach gripper to robot arm -->
